File: THB6064.brd (EAGLE design)
At the start: 59.1 x 43.2 mm, 30 parts, among them IC1 THB6064, J1 Inputs, J2 Motor, J3 MS1, J4 MS2, J5 MS3, J6 DCY1, J7 DCY2, J8 Power

Commit message: foo
Connections:
- net DIR: now also IC1.22, J1.4; no longer IC1.21, J1.3
- net STEP: now also IC1.21, J1.3; no longer IC1.22, J1.4
Routing:
- net STEP: track 39.0 -> 36.2 mm
- net DIR: track 36.2 -> 39.0 mm
- net MB-: track 59.7 -> 61.0 mm
- net MA+: track 59.7 -> 61.0 mm
- net +12V: track 70.2 -> 69.6 mm
