File: THB6064.sch (EAGLE design)
At the start: 30 parts, among them IC1 THB6064, J1 Inputs, J2 Motor, J3 MS1, J4 MS2, J5 MS3, J6 DCY1, J7 DCY2, J8 Power

Commit message: foo
Connections:
- net DIR: now also IC1.DIR, J1-4.1; no longer IC1.STEP, J1-3.1
- net STEP: now also IC1.STEP, J1-3.1; no longer IC1.DIR, J1-4.1
Changed lines of the file:
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@@
 <text x="73.66" y="127" size="1.27" layer="98">+5V</text>
 <text x="73.66" y="121.92" size="1.27" layer="98">Gnd</text>
-<text x="73.66" y="116.84" size="1.27" layer="98">Dir</text>
-<text x="73.66" y="111.76" size="1.27" layer="98">Step</text>
+<text x="73.66" y="111.76" size="1.27" layer="98">Dir</text>
+<text x="73.66" y="116.84" size="1.27" layer="98">Step</text>
 </plain>
 <instances>
@@
 <net name="DIR" class="0">
 <segment>
-<pinref part="J1" gate="-3" pin="1"/>
-<wire x1="88.9" y1="116.84" x2="93.98" y2="116.84" width="0.1524" layer="91"/>
-<wire x1="93.98" y1="116.84" x2="99.06" y2="111.76" width="0.1524" layer="91"/>
-<pinref part="IC1" gate="G$1" pin="STEP"/>
-<wire x1="99.06" y1="111.76" x2="137.16" y2="111.76" width="0.1524" layer="91"/>
-</segment>
-</net>
-<net name="STEP" class="0">
-<segment>
 <pinref part="J1" gate="-4" pin="1"/>
 <wire x1="88.9" y1="111.76" x2="96.52" y2="111.76" width="0.1524" layer="91"/>
@@
 </segment>
 </net>
+<net name="STEP" class="0">
+<segment>
+<pinref part="J1" gate="-3" pin="1"/>
+<wire x1="88.9" y1="116.84" x2="93.98" y2="116.84" width="0.1524" layer="91"/>
+<wire x1="93.98" y1="116.84" x2="99.06" y2="111.76" width="0.1524" layer="91"/>
+<pinref part="IC1" gate="G$1" pin="STEP"/>
+<wire x1="99.06" y1="111.76" x2="137.16" y2="111.76" width="0.1524" layer="91"/>
+</segment>
+</net>
